File: hardware/blueaudio-puck.kicad_sch (KiCad schematic)
At the start: 41 parts, among them J1 USB-C, J2 3.5mm, J3 OLED, J4 BATT, J5 PROG, SW1 MODE, SW2 RESET, U1 ESP32-WROOM-32U, U2 PCM5102A, U3 MCP73831-2-OT, U4 AP2112K-3.3, U5 LP2985-3.3

Commit message: hw: three user buttons, JLCPCB rules, and a router that models copper width
Brings the board in line with the three-button firmware, and fixes three
geometry bugs in the router that were producing copper which looked right and
was not.

Buttons. SW1/SW2/SW3 are now BT1/BT2/BT3 on GPIO 32/33/27, matching the
firmware; RESET and BOOT move to SW4/SW5. They sit in a row along the bottom
edge in the order a thumb expects -- previous, play, next. The board grew from
60x55 to 60x64 to make room: the old bottom edge was already full of headers,
and squeezing five switches into the sides would have put the two people press
constantly behind the headphone jack.

Worth recording: there is no LED on GPIO 27 on this board. The Kconfig help for
PUCK_LED_GPIO suggests 27 for an external status LED, which collides with BT3
on a breadboard. Here the only LED is D1 on CHG_STAT, so the pin is
unambiguously BT3.

JLCPCB rules are now in the project file, so DRC enforces them instead of
leaving them as folklore: 0.15 mm clearance, 0.2 mm track, 0.3 mm via drill,
0.13 mm annular ring, 0.5 mm hole-to-hole, 0.5 mm to the outline. Every value
sits at or inside their standard two-layer capability. Clearance is the only
one near a limit and is still 18% above their floor -- and the 0.05 mm it frees
per side against KiCad's 0.2 mm default is most of what lets the congested area
route at all. Teardrop parameters are configured too, though KiCad only
generates teardrops on demand, so they are a post-routing step rather than
something these files contain.

Three router bugs, each of which produced DRC-failing copper:

- A track is not a point. A 0.4 mm power track centred on a 0.25 mm grid cell
  spills into its neighbours, and checking only the cell it steps through let
  one sit 0.15 mm from a pad. Vias are worse: 0.6 mm across, and one landed on
  top of another net's track. Both now check every cell their copper covers.
- Clearance belongs in the check, not the map. Growing a clearance halo a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
Parts:
- added Q1, Q2: MMBT3904, Package_TO_SOT_SMD:SOT-23, symbol Transistor_BJT:MMBT3904
- added SW3: BT3, Button_Switch_SMD:Panasonic_EVQPUJ_EVQPUA, symbol Switch:SW_Push
- added SW4: RESET, Button_Switch_SMD:Panasonic_EVQPUJ_EVQPUA, symbol Switch:SW_Push
- added SW5: BOOT, Button_Switch_SMD:Panasonic_EVQPUJ_EVQPUA, symbol Switch:SW_Push
- SW1: value MODE -> BT1
- SW2: value RESET -> BT2
Connections:
- net +3V3: now also J5.2 (Pin_2); no longer J5.1 (Pin_1)
- net EN: now also Q1.3 (C), SW4.1; no longer J5.3 (Pin_3), SW2.1
- net GND: now also J5.1 (Pin_1), SW3.2, SW4.2, SW5.2; no longer J5.2 (Pin_2)
- net IO0: now also Q2.3 (C), SW5.1; no longer J5.4 (Pin_4)
- net RXD0: now also J5.3 (Pin_3); no longer J5.6 (Pin_6)
- net TXD0: now also J5.4 (Pin_4); no longer J5.5 (Pin_5)
- net BTN_3: now reaches U1.12 (IO27)
- net BTN_3: now also SW3.1
- net BTN_1: now reaches U1.8 (IO32)
- net BTN_1: now also SW1.1
- net BTN_MODE renamed BTN_2
- net BTN_2: now also SW2.1; no longer SW1.1
- new net DTR: J5.5 (Pin_5), Q1.2 (E), Q2.1 (B)
- new net RTS: J5.6 (Pin_6), Q1.1 (B), Q2.2 (E)
- no-connect marks 30 -> 28
Other:
- moved on the sheet: C1, C10, C11, C12, C13, C14, C15, C16, C17, C18, C2, C3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
